Commit message: edit structure

File: install/amr-gazebo-pkg/share/amr-gazebo-pkg/urdf/diffbot.urdf.xacro (robot description, xacro)
@@ -1 +1 @@
-/home/percy/camel-amr-projects/src/amr-gazebo-pkg/urdf/diffbot.urdf.xacro
+/home/sangjun/camel-amr-projects-UI/src/amr-gazebo-pkg/urdf/diffbot.urdf.xacro

File: src/amr-gazebo-pkg/urdf/diffbot_amr.urdf (robot description, URDF)
Before this commit: robot diffbot_amr, 8 links, 7 joints
Links:
- link chassis: geometry collision box size=.4 .2 .1; collision box size=1.1 .2 .1

File: src/amr-gazebo-pkg/urdf/diffbot_amr_obstacle.urdf (robot description, URDF)
Before this commit: robot diffbot_amr, 8 links, 7 joints
Links:
- link chassis: geometry collision box size=.4 .2 .1; collision box size=1.1 .2 .1
