Commit message: add data

File: src/amr-gazebo-pkg/urdf/diffbot.urdf.xacro (robot description, xacro)
@@ -152,5 +152,5 @@
       <origin xyz="0 0 0" rpy="0 0 0" />
       <geometry>
-        <box size="0.05 0.05 0.05"/>
+        <box size="0 0 0"/>
       </geometry>
     </visual>
@@ -158,5 +158,5 @@
       <origin xyz="0 0 0" rpy="0 0 0" />
       <geometry>
-        <box size="0.1 0.1 0.1"/>
+        <box size="0 0 0"/>
       </geometry>
     </collision>

File: src/amr-gazebo-pkg/urdf/diffbot_amr.urdf (robot description, URDF)
Before this commit: robot diffbot_amr, 9 links, 8 joints
Links:
- link chassis: geometry collision box size=.4 .2 .1; collision box size=1.1 .2 .025
