Commit message: added obstacle center calculation function

File: src/amr-gazebo-pkg/urdf/diffbot_amr.urdf (robot description, URDF)
Before this commit: robot diffbot_amr, 8 links, 7 joints
Links:
- link chassis: geometry collision box size=.4 .2 .1; collision box size=1.1 .2 .1

File: src/amr-gazebo-pkg/urdf/diffbot_amr_obstacle.urdf (robot description, URDF)
Before this commit: robot diffbot_amr, 8 links, 7 joints
Links:
- link chassis: geometry collision box size=.4 .2 .1; collision box size=1.1 .2 .1

Commit message: changed diffbot_amr.urdf (1*LiDAR >> 2*LiDAR, degree: 180 >> 270)

File: src/amr-gazebo-pkg/urdf/diffbot_amr.urdf (robot description, URDF)
Before this commit: robot diffbot_amr, 8 links, 7 joints
Links:
- added link hokuyo2, mass 1e-5; collision box size=0.05 0.05 0.05; visual box size=0.05 0.05 0.05
Joints:
- added joint hokuyo2_joint: type fixed, parent chassis, child hokuyo2, origin xyz=-0.455 0.325 0.18 rpy=0 0 3.141592, axis 0 1 0
- joint hokuyo_joint: origin xyz=0.555 0 0.13 rpy=0 0 0 -> xyz=0.455 -0.325 0.18 rpy=0 0 0

Commit message: ClusteringUpdate

File: src/amr-gazebo-pkg/urdf/diffbot_amr.urdf (robot description, URDF)
Before this commit: robot diffbot_amr, 9 links, 8 joints
Joints:
- joint hokuyo2_joint: origin xyz=-0.455 0.325 0.18 rpy=0 0 3.141592 -> xyz=-0.455 0.325 0.175 rpy=0 0 3.141592
- joint hokuyo_joint: origin xyz=0.455 -0.325 0.18 rpy=0 0 0 -> xyz=0.455 -0.325 0.175 rpy=0 0 0

Commit message: fixed LiDAR error (changed diffbot_amr.urdf)

File: src/amr-gazebo-pkg/urdf/diffbot_amr.urdf (robot description, URDF)
Before this commit: robot diffbot_amr, 9 links, 8 joints
Joints:
- joint hokuyo2_joint: origin xyz=-0.455 0.325 0.18 rpy=0 0 3.141592 -> xyz=-0.55 0.45 0.171 rpy=0 0 3.141592
- joint hokuyo_joint: origin xyz=0.455 -0.325 0.18 rpy=0 0 0 -> xyz=0.55 -0.45 0.171 rpy=0 0 0

Commit message: a

File: src/amr-gazebo-pkg/urdf/diffbot_amr.urdf (robot description, URDF)
Before this commit: robot diffbot_amr, 9 links, 8 joints
Links:
- link chassis: geometry collision box size=.4 .2 .1; collision box size=1.1 .2 .1
Joints:
- joint hokuyo2_joint: origin xyz=-0.455 0.325 0.175 rpy=0 0 3.141592 -> xyz=-0.55 0.45 0.171 rpy=0 0 3.141592
- joint hokuyo_joint: origin xyz=0.455 -0.325 0.175 rpy=0 0 0 -> xyz=0.55 -0.45 0.171 rpy=0 0 0

Commit message: updated UI

File: src/amr-gazebo-pkg/urdf/diffbot_amr.urdf (robot description, URDF)
Before this commit: robot diffbot_amr, 9 links, 8 joints
Links:
- link chassis: geometry collision box size=.4 .2 .1; collision box size=1.1 .2 .1
Joints:
- joint hokuyo2_joint: origin xyz=-0.455 0.325 0.175 rpy=0 0 3.141592 -> xyz=-0.55 0.45 0.171 rpy=0 0 3.141592
- joint hokuyo_joint: origin xyz=0.455 -0.325 0.175 rpy=0 0 0 -> xyz=0.55 -0.45 0.171 rpy=0 0 0

File: src/amr-gazebo-pkg/urdf/diffbot_amr_obstacle.urdf (robot description, URDF)
Before this commit: robot diffbot_amr, 8 links, 7 joints
Links:
- link chassis: geometry collision box size=.4 .2 .1; collision box size=1.1 .2 .1
